File: JuiceAdapter.kicad_pcb (KiCad board)
At the start: 2 copper layers, 24 x 10 mm, 6 parts, among them J1 Conn_01x04_Pin, J2 Conn_01x04_Pin, Q1 MMDT5401

Commit message: Clarified resistor values on schematic and PCB.
Parts:
- R1, R2: value R -> 2.4KΩ
- R3: value R -> 75Ω
Changed lines of the file:
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@@
 			)
 		)
-		(property "Value" "R"
-			(at -1 -3.2 0)
+		(property "Value" "75Ω"
+			(at -1.09 -3.5 0)
 			(layer "F.Fab")
 			(effects
@@
 			)
 		)
-		(property "Description" "Resistor"
+		(property "Description" "Resistor - 75Ohm"
 			(at 0 0 0)
 			(unlocked yes)
@@
 		)
 		(fp_text user "${REFERENCE}"
-			(at -1 -4.2 0)
+			(at -1 -4.74 0)
 			(layer "F.Fab")
 			(effects
@@
 			)
 		)
-		(property "Value" "R"
-			(at 0.4 -3.1 0)
+		(property "Value" "2.4KΩ"
+			(at 0.38 -3.5 0)
 			(layer "F.Fab")
 			(effects
@@
 			)
 		)
-		(property "Description" "Resistor"
+		(property "Description" "Resistor - 2.4kOhm"
 			(at 0 0 0)
 			(unlocked yes)
@@
 			)
 		)
-		(property "LCSC PN" "C304065"
+		(property "LCSC PN" "C22940  "
 			(at 0 0 0)
 			(unlocked yes)
@@
 		)
 		(fp_text user "${REFERENCE}"
-			(at 0.4 -4.2 0)
+			(at 0.45 -4.63 0)
 			(layer "F.Fab")
 			(effects
@@
 			)
 		)
-		(property "Value" "R"
+		(property "Value" "2.4KΩ"
 			(at -5.4 0.7 180)
 			(layer "F.Fab")
@@
 			)
 		)
-		(property "Description" "Resistor"
+		(property "Description" "Resistor - 2.4kOhm"
 			(at 0 0 90)
 			(unlocked yes)
@@
 			)
 		)
-		(property "LCSC PN" "C304065"
+		(property "LCSC PN" "C22940  "
 			(at 0 0 90)
 			(unlocked yes)
